File: clkdiv2.kicad_sch (KiCad schematic)
At the start: 40 parts, among them J1 Conn_02x05_Odd_Even, Q1 BC847, Q2 BC847, Q3 BC847, SW1 SW_Rotary12, U1 4017

Commit message: pcb ready for v0 manu
Parts:
- added H5: in, Eurorack:Mech-AudioJack-Hole-Input-Clock, symbol Mechanical:MountingHole_Pad
- added H6: reset, Eurorack:Mech-AudioJack-Hole-Input-Gate, symbol Mechanical:MountingHole_Pad
- added H7: out, Eurorack:Mech-AudioJack-Hole-Output-Gate, symbol Mechanical:MountingHole_Pad
- added H8: step, Eurorack:Mech-MRK-Hole, symbol Mechanical:MountingHole_Pad
- added H9: led, Eurorack:Mech-LED-Hole-3mm-Bezel, symbol Mechanical:MountingHole_Pad
- added J10, J6, J8: Conn_01x03_Pin, Connector_PinHeader_2.54mm:PinHeader_1x03_P2.54mm_Vertical, symbol Connector:Conn_01x03_Pin
- added J2, J3, J4: AudioJack2_SwitchT, Eurorack:AudioJack2_Tayda_A-2566, symbol Eurorack:AudioJack2_SwitchT
- added J5, J7, J9: Conn_01x03_Socket, Connector_PinSocket_2.54mm:PinSocket_1x03_P2.54mm_Vertical, symbol Connector:Conn_01x03_Socket
- added R17: 120K, Resistor_SMD:R_0805_2012Metric, symbol Device:R
- added R18, R19: 1K, Resistor_SMD:R_0805_2012Metric, symbol Device:R
- added R20: 10, Resistor_SMD:R_0805_2012Metric, symbol Device:R
- C3: footprint (none) -> Capacitor_SMD:C_0805_2012Metric
- C4: footprint (none) -> Capacitor_THT:C_Rect_L7.2mm_W2.5mm_P5.00mm_FKS2_FKP2_MKS2_MKP2
- D10: footprint (none) -> LED_THT:LED_D3.0mm
- D3, D4, D5, D6, D7, D8: footprint (none) -> Diode_SMD:D_SOD-323_HandSoldering
- D9: value 5.1V -> Zener 5.1V; footprint (none) -> Diode_SMD:D_MiniMELF
- Q1, Q2, Q3: footprint (none) -> Package_SO:TSOP-6_1.65x3.05mm_P0.95mm; PartNum (none) -> 771-BCM847DS135; Vendor (none) -> Mouser
- R10, R11, R12, R13, R3, R5, R6, R7, R8, R9: footprint (none) -> Resistor_SMD:R_0805_2012Metric
- R14: value 20K -> 22K; footprint (none) -> Resistor_SMD:R_0805_2012Metric
- R15: value 100K -> 4.7K; footprint (none) -> Resistor_SMD:R_0805_2012Metric
- R16: value 1K -> 220K; footprint (none) -> Resistor_SMD:R_0805_2012Metric
- R4: value 1M -> 1.2M; footprint (none) -> Resistor_SMD:R_0805_2012Metric
- SW1: footprint (none) -> Eurorack:Switch_Rotary_NKK_MRK_112; PartNum (none) -> 633-MRK112-BA; Vendor (none) -> Mouser
- U1: footprint (none) -> Package_SO:TSSOP-16_4.4x5mm_P0.65mm; PartNum (none) -> 595-CD4017BPWR; Vendor (none) -> Mouser
Connections:
- net +12V: now also J5.1 (Pin_1), R20.1; no longer C3.1, Q3.1 (C2), Q3.3 (C1), U1.16 (VDD)
- net -12V: no longer C2.2
- net FACE: now also H5.1, H6.1, H7.1, H8.1, H9.1
- net GND: now also J5.2 (Pin_2); no longer C3.2, D9.2 (A), R15.2, R16.1, U1.13 (CKEN), U1.8 (VSS)
- net IN: now also J9.1 (Pin_1)
- net OUT: now also J4.T, R18.1; no longer D9.1 (K), R14.2, R15.1
- net RST: now also J9.2 (Pin_2)
- net _IN: now reaches Q1.3 (C2), R6.1
- net _IN: now also J7.1 (Pin_1); no longer D6.1 (K), U1.14 (CLK)
- net at D6.2 (A), D7.2 (A): now also R14.2, R15.1; no longer Q3.5 (B1), Q3.6 (B2)
- net at Q3.4 (E1): now also D9.1 (K), R17.1, R18.2; no longer R14.1
- net _RST: now reaches D5.1 (K), R13.1
- net _RST: now also J7.2 (Pin_2); no longer D8.1 (K), U1.15 (Reset)
- net at D10.1 (K): now also R19.2; no longer R16.2
- new net: Q3.5 (B1), Q3.6 (B2), R15.2, R16.2
- new net 12V': C3.1, J6.1 (Pin_1), R14.1, U1.16 (VDD)
- new net GND': C3.2, D9.2 (A), J2.S, J3.S, J4.S, J6.2 (Pin_2), R16.1, R17.2, R19.1, U1.13 (CKEN), U1.8 (VSS)
- new net IN': J10.1 (Pin_1), J2.T
- new net RST': J10.2 (Pin_2), J3.T
- new net V_LED: C2.2, J5.3 (Pin_3), R20.2
- new net V_LED': J6.3 (Pin_3), Q3.1 (C2), Q3.3 (C1)
- new net _IN': D6.1 (K), J8.1 (Pin_1), U1.14 (CLK)
- new net _RST': D8.1 (K), J8.2 (Pin_2), U1.15 (Reset)
- no-connect marks 4 -> 11
Other:
- moved on the sheet: C3, C4, D10, D4, D5, D6, D7, D8, D9, Q2A, Q2B, Q3A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

Commit message: pcb ready for v0a manu
Parts:
- removed Q3: BC847, Package_SO:TSOP-6_1.65x3.05mm_P0.95mm, symbol Device:Q_Dual_NPN_NPN_C2E2C1E1B1B2
- added Q3: BCM847, Package_SO:TSOP-6_1.65x3.05mm_P0.95mm, symbol Device:Q_Dual_NPN_NPN_E1B1C2E2B2C1
- Q1, Q2: value BC847 -> BCM847
Connections:
- net V_LED': now also Q3.3 (C2), Q3.6 (C1)
- net at D9.1 (K), R17.1, R18.2: now also Q3.4 (E2)
- net at R15.2, R16.2: now also Q3.2 (B1), Q3.5 (B2)
- net at D10.2 (A): now also Q3.1 (E1)
Changed lines of the file:
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@@
       (effects (font (size 1.27 1.27)) (justify left))
     )
-    (property "Value" "BC847" (at 116.84 95.25 0)
+    (property "Value" "BCM847" (at 116.84 95.25 0)
       (effects (font (size 1.27 1.27)) (justify left))
     )
@@
       (effects (font (size 1.27 1.27)) (justify left))
     )
-    (property "Value" "BC847" (at 88.9 55.88 0)
+    (property "Value" "BCM847" (at 88.9 55.88 0)
       (effects (font (size 1.27 1.27)) (justify left))
     )
@@
       (effects (font (size 1.27 1.27)) (justify left))
     )
-    (property "Value" "BC847" (at 90.17 100.33 0)
+    (property "Value" "BCM847" (at 90.17 100.33 0)
       (effects (font (size 1.27 1.27)) (justify left))
     )
@@
       (effects (font (size 1.27 1.27)) (justify left))
     )
-    (property "Value" "BC847" (at 109.22 50.8 0)
+    (property "Value" "BCM847" (at 109.22 50.8 0)
       (effects (font (size 1.27 1.27)) (justify left))
     )
@@
         (path "/54607e40-577c-4def-b17c-96859aef0795"
           (reference "#PWR010") (unit 1)
-        )
-      )
-    )
-  )
-  (symbol (lib_id "Device:Q_Dual_NPN_NPN_C2E2C1E1B1B2") (at 248.92 55.88 0) (unit 2)
-    (in_bom yes) (on_board yes) (dnp no) (fields_autoplaced)
-    (property "Reference" "Q3" (at 254 54.61 0)
-      (effects (font (size 1.27 1.27)) (justify left))
-    )
-    (property "Value" "BC847" (at 254 57.15 0)
-      (effects (font (size 1.27 1.27)) (justify left))
-    )
-    (property "Footprint" "Package_SO:TSOP-6_1.65x3.05mm_P0.95mm" (at 254 53.34 0)
-      (effects (font (size 1.27 1.27)) hide)
-    )
-    (property "Datasheet" "~" (at 248.92 55.88 0)
-      (effects (font (size 1.27 1.27)) hide)
-    )
-    (property "Vendor" "Mouser" (at 248.92 55.88 0)
-      (effects (font (size 1.27 1.27)) hide)
-    )
-    (property "PartNum" "771-BCM847DS135" (at 248.92 55.88 0)
-      (effects (font (size 1.27 1.27)) hide)
-    )
-    (pin "6")
-    (pin "3")
-    (pin "1")
-    (pin "5")
-    (pin "4")
-    (pin "2")
-    (instances
-      (project "clkdiv2"
-        (path "/54607e40-577c-4def-b17c-96859aef0795"
-          (reference "Q3") (unit 2)
         )
       )
@@
     )
   )
+  (symbol (lib_id "Device:Q_Dual_NPN_NPN_E1B1C2E2B2C1") (at 238.76 27.94 0) (unit 2)
+    (in_bom yes) (on_board yes) (dnp no) (fields_autoplaced)
+    (property "Reference" "Q3" (at 243.84 26.67 0)
+      (effects (font (size 1.27 1.27)) (justify left))
+    )
+    (property "Value" "BCM847" (at 243.84 29.21 0)
+      (effects (font (size 1.27 1.27)) (justify left))
+    )
+    (property "Footprint" "Package_SO:TSOP-6_1.65x3.05mm_P0.95mm" (at 243.84 25.4 0)
+      (effects (font (size 1.27 1.27)) hide)
+    )
+    (property "Datasheet" "~" (at 238.76 27.94 0)
+      (effects (font (size 1.27 1.27)) hide)
+    )
+    (property "Vendor" "Mouser" (at 238.76 27.94 0)
+      (effects (font (size 1.27 1.27)) hide)
+    )
+    (property "PartNum" "771-BCM847DS135" (at 238.76 27.94 0)
+      (effects (font (size 1.27 1.27)) hide)
+    )
+    (pin "6")
+    (pin "1")
+    (pin "5")
+    (pin "2")
+    (pin "4")
+    (pin "3")
+    (instances
+      (project "clkdiv2"
+        (path "/54607e40-577c-4def-b17c-96859aef0795"
+          (reference "Q3") (unit 2)
+        )
+      )
+    )
+  )
   (symbol (lib_id "power:GND") (at 106.68 116.84 0) (unit 1)
     (in_bom yes) (on_board yes) (dnp no) (fields_autoplaced)
@@
     )
   )
-  (symbol (lib_id "Device:Q_Dual_NPN_NPN_C2E2C1E1B1B2") (at 238.76 27.94 0) (unit 1)
-    (in_bom yes) (on_board yes) (dnp no) (fields_autoplaced)
-    (property "Reference" "Q3" (at 243.84 26.67 0)
-      (effects (font (size 1.27 1.27)) (justify left))
-    )
-    (property "Value" "BC847" (at 243.84 29.21 0)
-      (effects (font (size 1.27 1.27)) (justify left))
-    )
-    (property "Footprint" "Package_SO:TSOP-6_1.65x3.05mm_P0.95mm" (at 243.84 25.4 0)
-      (effects (font (size 1.27 1.27)) hide)
-    )
-    (property "Datasheet" "~" (at 238.76 27.94 0)
-      (effects (font (size 1.27 1.27)) hide)
-    )
-    (property "Vendor" "Mouser" (at 238.76 27.94 0)
-      (effects (font (size 1.27 1.27)) hide)
-    )
-    (property "PartNum" "771-BCM847DS135" (at 238.76 27.94 0)
-      (effects (font (size 1.27 1.27)) hide)
-    )
-    (pin "6")
-    (pin "3")
-    (pin "1")
-    (pin "5")
-    (pin "4")
-    (pin "2")
-    (instances
-      (project "clkdiv2"
-        (path "/54607e40-577c-4def-b17c-96859aef0795"
-          (reference "Q3") (unit 1)
-        )
-      )
-    )
-  )
   (symbol (lib_id "Mechanical:MountingHole_Pad") (at 33.02 177.8 0) (unit 1)
     (in_bom no) (on_board yes) (dnp no) (fields_autoplaced)
@@
         )
       )
+    )
+  )
+  (symbol (lib_id "Device:Q_Dual_NPN_NPN_E1B1C2E2B2C1") (at 248.92 55.88 0) (unit 1)
+    (in_bom yes) (on_board yes) (dnp no) (fields_autoplaced)
+    (property "Reference" "Q3" (at 254 54.61 0)
+      (effects (font (size 1.27 1.27)) (justify left))
+    )
+    (property "Value" "BCM847" (at 254 57.15 0)
+      (effects (font (size 1.27 1.27)) (justify left))
+    )
+    (property "Footprint" "Package_SO:TSOP-6_1.65x3.05mm_P0.95mm" (at 254 53.34 0)
+      (effects (font (size 1.27 1.27)) hide)
+    )
+    (property "Datasheet" "~" (at 248.92 55.88 0)
+      (effects (font (size 1.27 1.27)) hide)
+    )
+    (property "Vendor" "Mouser" (at 248.92 55.88 0)
+      (effects (font (size 1.27 1.27)) hide)
+    )
+    (property "PartNum" "771-BCM847DS135" (at 248.92 55.88 0)
+      (effects (font (size 1.27 1.27)) hide)
+    )
+    (pin "6")
+    (pin "1")
+    (pin "5")
+    (pin "2")
+    (pin "4")
+    (pin "3")
+    (instances
+      (project "clkdiv2"
+        (path "/54607e40-577c-4def-b17c-96859aef0795"
+          (reference "Q3") (unit 1)
+        )
+      )
